Commit message: Commit inicial

File: wamv_gazebo/urdf/components/lidar.xacro (robot description, xacro)
@@ -5,7 +5,7 @@
                params = "type:='16_beam'
                          name
-                         x:=0.7 y:=0 z:=1.8
+                         x:=0 y:=0 z:=0
                          R:=0 P:=0 Y:=0
-                         post_Y:=0 post_z_from:=1.2965">
+                         post_Y:=0 post_z_from:=0">
     <xacro:if value="${type == '16_beam'}">
       <xacro:wamv_3d_lidar name="${name}"

File: wamv_gazebo/urdf/components/wamv_camera.xacro (robot description, xacro)
@@ -1,5 +1,5 @@
 <?xml version="1.0"?>
 <robot xmlns:xacro="http://ros.org/wiki/xacro">
-  <xacro:macro name="wamv_camera" params="name x:=0.5 y:=0 z:=1.5 post_z_from:=1.2965 R:=0 P:=0 Y:=0 post_Y:=0 visualize:=False">
+  <xacro:macro name="wamv_camera" params="name x:=0.5 y:=0 z:=1.5 post_z_from:=0.2 R:=0 P:=0 Y:=0 post_Y:=0 visualize:=False">
     <!-- Define length variables for link positioning -->
     <xacro:property name="platform_z" value="${post_z_from}"/>

File: wamv_gazebo/urdf/components/wamv_gps.xacro (robot description, xacro)
@@ -1,5 +1,6 @@
 <?xml version="1.0" encoding="UTF-8"?>
 <robot xmlns:xacro="http://ros.org/wiki/xacro">
-  <xacro:macro name="wamv_gps" params="name:=gps x:=0.3 y:=0 z:=1.3
+  <xacro:macro name="wamv_gps" params="name:=gps x:=0.4 y:=0 z:=0.55
+  					lat:=21.30996 lon:=-157.8901 elev:=0.0
 				       R:=0 P:=0 Y:=0 update_rate:=15">
     <link name="${namespace}/${name}_link">

File: wamv_gazebo/urdf/macros.xacro (robot description, xacro)
@@ -14,5 +14,3 @@
   <xacro:include filename="$(find wamv_gazebo)/urdf/components/wamv_p3d.xacro" />
   <xacro:include filename="$(find wamv_gazebo)/urdf/components/wamv_pinger.xacro" />
-  <!-- Include ball shooter macros -->
-  <xacro:include filename="$(find wamv_gazebo)/urdf/components/ball_shooter.xacro" />
 </robot>

File: wamv_gazebo/urdf/thruster_layouts/wamv_aft_thrusters.xacro (robot description, xacro)
@@ -7,5 +7,4 @@
     <plugin name="wamv_gazebo_thrust" filename="libusv_gazebo_thrust_plugin.so">
       <cmdTimeout>1.0</cmdTimeout>
-      <publisherRate>100.0</publisherRate>
       <robotNamespace>${namespace}</robotNamespace>
       <xacro:include filename="$(find wamv_gazebo)/urdf/thruster_layouts/wamv_gazebo_thruster_config.xacro" />

File: wamv_gazebo/urdf/thruster_layouts/wamv_gazebo_thruster_config.xacro (robot description, xacro)
@@ -13,6 +13,6 @@
       <mappingType>1</mappingType>
       <maxCmd>1.0</maxCmd>
-      <maxForceFwd>250.0</maxForceFwd>
-      <maxForceRev>-100.0</maxForceRev>
+      <maxForceFwd>2.5</maxForceFwd>
+      <maxForceRev>-2.5</maxForceRev>
       <maxAngle>${pi/2}</maxAngle>
     </thruster>

File: wamv_gazebo/urdf/thruster_layouts/wamv_t_thrusters.xacro (robot description, xacro)
@@ -2,11 +2,10 @@
 <robot xmlns:xacro="http://ros.org/wiki/xacro">
   <xacro:include filename="$(find wamv_description)/urdf/thrusters/engine.xacro" />
-  <xacro:engine prefix="left" position="-2.373776 1.027135 0.318237" />
-  <xacro:engine prefix="right" position="-2.373776 -1.027135 0.318237" />
-  <xacro:engine prefix="lateral" position="0.0 0.0 0.318237" orientation="0.0 0.0 1.5707"/>
+  <xacro:engine prefix="left" position="${0.95+0.38} ${0.33} 0.368237" orientation="0.0 0.0 0.0" />
+  <xacro:engine prefix="right" position="${0.95+0.38} ${-0.33} 0.368237"  orientation="0.0 0.0 0.0" />
+  <xacro:engine prefix="lateral" position="${0.68} ${0} 0.265237" orientation="0.0 0.0 0.0"/>
   <gazebo>
     <plugin name="wamv_gazebo_thrust" filename="libusv_gazebo_thrust_plugin.so">
       <cmdTimeout>1.0</cmdTimeout>
-      <publisherRate>100.0</publisherRate>
       <robotNamespace>${namespace}</robotNamespace>
       <xacro:include filename="$(find wamv_gazebo)/urdf/thruster_layouts/wamv_gazebo_thruster_config.xacro" />

File: wamv_gazebo/urdf/thruster_layouts/wamv_x_thrusters.xacro (robot description, xacro)
@@ -9,5 +9,4 @@
     <plugin name="wamv_gazebo_thrust" filename="libusv_gazebo_thrust_plugin.so">
       <cmdTimeout>1.0</cmdTimeout>
-      <publisherRate>100.0</publisherRate>
       <robotNamespace>${namespace}</robotNamespace>
       <xacro:include filename="$(find wamv_gazebo)/urdf/thruster_layouts/wamv_gazebo_thruster_config.xacro" />

File: wamv_gazebo/urdf/wamv_gazebo.urdf.xacro (robot description, xacro)
@@ -5,12 +5,13 @@
   <xacro:arg name="locked" default="false" />
   <xacro:arg name="thruster_config" default="H" />
-  <xacro:arg name="camera_enabled" default="false" />
-  <xacro:arg name="gps_enabled" default="false" />
-  <xacro:arg name="imu_enabled" default="false" />
-  <xacro:arg name="lidar_enabled" default="false" />
+  <xacro:arg name="camera_enabled" default="true" />
+  <xacro:arg name="gps_enabled" default="true" />
+  <xacro:arg name="imu_enabled" default="true" />
+  <xacro:arg name="lidar_enabled" default="true" />
+  <xacro:arg name="planar_enabled" default="true" />
+  <xacro:arg name="sonar_enabled" default="true" />
   <xacro:arg name="ground_truth_enabled" default="false" />
   <xacro:arg name="vrx_sensors_enabled" default="false" />
   <xacro:arg name="pinger_enabled" default="false" />
-  <xacro:arg name="ball_shooter_enabled" default="false" />
   <xacro:arg name="thruster_namespace" default="thrusters/"/>
   <xacro:arg name="camera_namespace" default="cameras/"/>
@@ -35,8 +36,4 @@
   <!-- === The WAM-V platform === -->
   <xacro:include filename="$(find wamv_gazebo)/urdf/wamv_gazebo.xacro"/>
-  <!-- === Batteries === -->
-  <xacro:include filename="$(find wamv_description)/urdf/battery.xacro"/>
-  <xacro:battery prefix="left" position="0 1 0.45" orientation="0 0 0"/>
-  <xacro:battery prefix="right" position="0 -1 0.45" orientation="0 0 0"/>
   <!-- === Thrusters === -->
   <!-- Use thruster yaml file if given -->
@@ -92,17 +89,24 @@
     <xacro:include filename="$(arg component_xacro_file)"/>
     <xacro:yaml_components />
+    <!-- sonar_enabled -->
+      <xacro:if value="$(arg sonar_enabled)">
+    <xacro:sonar name="sonar_sensor" x="1.6" y="0.4" z="0.6" ros_topic="/distance1" Y="${radians(0)}"  update_rate="10" min_range="0.3" max_range="2" field_of_view="56" ray_count="2" />
+    <xacro:sonar name="sonar_sensor2" x="1.6" y="-0.4" z="0.6" ros_topic="/distance2" Y="${radians(0)}" update_rate="10" min_range="0.3" max_range="2" field_of_view="56" ray_count="2" />
+    <xacro:sonar name="sonar_sensor3" x="0.3" y="0.4" z="0.6" ros_topic="/distance3" Y="${radians(180)}" update_rate="10" min_range="0.3" max_range="2" field_of_view="56" ray_count="2" />
+    <xacro:sonar name="sonar_sensor4" x="0.3" y="-0.4" z="0.6" ros_topic="/distance4" Y="${radians(180)}" update_rate="10" min_range="0.3" max_range="2" field_of_view="56" ray_count="2" />
+  </xacro:if>
     <!-- Add CPU Cases -->
     <xacro:include filename="$(find wamv_description)/urdf/cpu_cases.xacro" />
-    <xacro:cpu_cases position="-0.15 0 1.53" orientation="0 0 0"/>
+    <xacro:cpu_cases position="0.75 0 0.65" orientation="0 0 0"/>
   </xacro:if>
   <!-- Otherwise, add sensors based on enable variables -->
   <xacro:unless value="$(arg yaml_component_generation)">
-    <!-- Add a front camera -->
+    <!-- Add a front camera
     <xacro:if value="$(arg camera_enabled)">
-      <xacro:wamv_camera name="front_camera" y="0.3" x="0.75" P="${radians(15)}" />
-    </xacro:if>
+      <xacro:wamv_camera name="front_camera" y="0" x="1.5" z="0.65" P="${radians(-20)}" />
+    </xacro:if>-->
     <!-- Add simulated GPS -->
     <xacro:if value="$(arg gps_enabled)">
-      <xacro:wamv_gps name="gps_wamv" x="-0.85" />
+      <xacro:wamv_gps name="gps_wamv" x="0.4" y="0" z="0.55" />
     </xacro:if>
     <!-- Add Simulated IMU -->
@@ -112,6 +116,10 @@
     <!-- Add 3D LIDAR -->
     <xacro:if value="$(arg lidar_enabled)">
-      <xacro:lidar name="lidar_wamv" y="-0.3" type="16_beam"/>
+      <xacro:lidar name="lidar_wamv" x="0.8" y="0" z="0.7" type="16_beam"/>
     </xacro:if>
+      <!-- Add PLANAR -->
+  	<xacro:if value="$(arg planar_enabled)">
+    	<xacro:wamv_multibeam_laser name="planar_wamv" x="1.2" y="0" z="1"/>
+  	</xacro:if>
     <!-- Add P3D ground truth -->
     <xacro:if value="$(arg ground_truth_enabled)">
@@ -122,28 +130,16 @@
       <xacro:wamv_pinger name="pinger" position="1.0 0 -1.0" />
     </xacro:if>
-    <!-- Add ball shooter (default pitch angle: ~-60 deg) -->
-    <xacro:if value="$(arg ball_shooter_enabled)">
-      <xacro:wamv_ball_shooter name="ball_shooter" x="0.54" y="0.30" z="1.296" pitch="-1.04"/>
-    </xacro:if>
     <!-- ==== VRX sensor configuration ==== -->
     <xacro:if value="$(arg vrx_sensors_enabled)">
       <!-- Add CPU Cases -->
       <xacro:include filename="$(find wamv_description)/urdf/cpu_cases.xacro" />
-      <xacro:cpu_cases position="-0.15 0 1.53" orientation="0 0 0"/>
+      <xacro:cpu_cases position="0.75 0 0.65" orientation="0 0 0"/>
       <!-- Add a stereo camera pair -->
-      <xacro:wamv_camera name="front_left_camera" y="0.1" x="0.75" P="${radians(15)}" />
-      <xacro:wamv_camera name="front_right_camera" y="-0.1" x="0.75" P="${radians(15)}" />
+     <!-- <xacro:wamv_camera name="front_left_camera" y="0.1" x="0.75" P="${radians(15)}" />-->
+      <!--<xacro:wamv_camera name="front_right_camera" y="-0.1" x="0.75" P="${radians(15)}" />-->
       <!-- Add a camera facing right -->
-      <xacro:wamv_camera name="middle_right_camera" y="-0.45" P="${radians(15)}" Y="${radians(-90)}" post_Y="${radians(-90)}" />
-      <!-- Add simulated GPS -->
-      <xacro:wamv_gps name="gps_wamv" x="-0.85" />
-      <!-- Add Simulated IMU -->
-      <xacro:wamv_imu name="imu_wamv" y="-0.2" />
-      <!-- Add 3D LIDAR -->
-      <xacro:lidar name="lidar_wamv" type="16_beam"/>
-      <!-- Add pinger -->
-      <xacro:wamv_pinger name="pinger" position="1.0 0 -1.0" />
-      <!-- Add ball shooter (default pitch angle: ~-60 deg) -->
-      <xacro:wamv_ball_shooter name="ball_shooter" x="0.54" y="0.30" z="1.296" pitch="-1.04"/>
+      <xacro:if value="$(arg camera_enabled)">
+      <xacro:wamv_camera name="middle_right_camera" y="0" x="1.5" z="0.65" />
+    </xacro:if>
     </xacro:if>
   </xacro:unless>
