Commit message: Commit segundo

File: wamv_description/urdf/thrusters/engine.xacro (robot description, xacro)
@@ -4,4 +4,5 @@
   <xacro:macro name="engine" params="prefix position:='0 0 0' orientation:='0 0 0'">
     <link name="${namespace}/${prefix}_engine_link">
+    <!--
       <visual>
         <geometry>
@@ -9,4 +10,5 @@
         </geometry>
       </visual>
+       -->
       <collision name="${prefix}_engine_vertical_axis_collision">
         <origin xyz="-0.16 0 -0.24" rpy="0 0 0" />
@@ -22,5 +24,5 @@
       </collision>
       <inertial>
-        <mass value="15"/>
+        <mass value="0.1"/>
         <inertia ixx="0.889245" ixy="0.0" ixz="0.0" iyy="0.911125" iyz="0.0" izz="0.078125"/>
       </inertial>
@@ -33,5 +35,5 @@
       </visual>
       <collision name="${prefix}_propeller_collision">
-        <origin xyz="-0.08 0 0" rpy="0 1.57 0" />
+        <origin xyz="0 0 0" rpy="0 1.57 0" />
         <geometry>
           <cylinder length="0.18" radius="0.24" />
@@ -39,5 +41,5 @@
       </collision>
       <inertial>
-        <mass value="0.5"/>
+        <mass value="0.05"/>
         <inertia ixx="0.008545" ixy="0.0" ixz="0.0" iyy="0.008545" iyz="0.0" izz="0.0144"/>
       </inertial>

File: wamv_description/urdf/wamv_base.urdf.xacro (robot description, xacro)
@@ -1,7 +1,4 @@
 <?xml version="1.0"?>
 <robot xmlns:xacro="http://ros.org/wiki/xacro" name="wam-v">
-  <!-- Required arg for melodic and kinetic... -->
-  <xacro:arg name="namespace" default="wamv"/>
-  <xacro:property name="namespace" value="$(arg namespace)" scope="global" />
   <!-- Macro for creating the main collisions as simple shapes. -->
   <xacro:macro name="main_collisions" params="prefix reflect:=1">

File: wamv_gazebo/urdf/components/wamv_3d_lidar.xacro (robot description, xacro)
@@ -68,5 +68,5 @@
       <visual>
         <geometry>
-          <cylinder radius="${post_radius}" length="${post_length}"/>
+          <cylinder radius="0" length="0"/>
         </geometry>
         <material name="${name}_post_material">
@@ -76,5 +76,5 @@
       <collision name="${name}_post_collision">
         <geometry>
-          <cylinder radius="${post_radius}" length="${post_length}"/>
+          <cylinder radius="0" length="0"/>
         </geometry>
       </collision>
@@ -82,7 +82,7 @@
         <mass value="${post_mass}"/>
         <inertia
-          ixx="${(post_mass/12) * (3*post_radius*post_radius + post_length*post_length)}"
-          iyy="${(post_mass/12) * (3*post_radius*post_radius + post_length*post_length)}"
-          izz="${(post_mass/2) * (post_radius*post_radius)}"
+          ixx="0"
+          iyy="0"
+          izz="0"
           ixy="0"
           ixz="0"

File: wamv_gazebo/urdf/components/wamv_camera.xacro (robot description, xacro)
@@ -52,5 +52,5 @@
       <visual>
         <geometry>
-          <cylinder radius="${post_radius}" length="${post_length}"/>
+          <cylinder radius="0" length="0"/>
         </geometry>
         <material name="${name}_post_material">
@@ -60,5 +60,5 @@
       <collision name="${name}_post_collision">
         <geometry>
-          <cylinder radius="${post_radius}" length="${post_length}"/>
+          <cylinder radius="0" length="0"/>
         </geometry>
       </collision>
@@ -66,7 +66,7 @@
         <mass value="${post_mass}"/>
         <inertia
-          ixx="${(post_mass/12) * (3*post_radius*post_radius + post_length*post_length)}"
-          iyy="${(post_mass/12) * (3*post_radius*post_radius + post_length*post_length)}"
-          izz="${(post_mass/2) * (post_radius*post_radius)}"
+          ixx="0"
+          iyy="0"
+          izz="0"
           ixy="0"
           ixz="0"

File: wamv_gazebo/urdf/macros.xacro (robot description, xacro)
@@ -14,3 +14,4 @@
   <xacro:include filename="$(find wamv_gazebo)/urdf/components/wamv_p3d.xacro" />
   <xacro:include filename="$(find wamv_gazebo)/urdf/components/wamv_pinger.xacro" />
+  <xacro:include filename="$(find wamv_gazebo)/urdf/components/sonar_sensor.xacro" />
 </robot>

File: wamv_gazebo/urdf/wamv_gazebo.urdf.xacro (robot description, xacro)
@@ -11,11 +11,8 @@
   <xacro:arg name="planar_enabled" default="true" />
   <xacro:arg name="sonar_enabled" default="true" />
-  <xacro:arg name="ground_truth_enabled" default="false" />
   <xacro:arg name="vrx_sensors_enabled" default="false" />
-  <xacro:arg name="pinger_enabled" default="false" />
   <xacro:arg name="thruster_namespace" default="thrusters/"/>
   <xacro:arg name="camera_namespace" default="cameras/"/>
   <xacro:arg name="sensor_namespace" default="sensors/"/>
-  <xacro:arg name="pinger_namespace" default="pingers/"/>
   <xacro:arg name="shooter_namespace" default="shooters/"/>
   <!-- Note: this is only used for some sensors that do not correctly use the
@@ -25,5 +22,4 @@
   <xacro:property name="camera_namespace" value="$(arg camera_namespace)" scope="global" />
   <xacro:property name="sensor_namespace" value="$(arg sensor_namespace)" scope="global" />
-  <xacro:property name="pinger_namespace" value="$(arg pinger_namespace)" scope="global" />
   <xacro:property name="shooter_namespace" value="$(arg shooter_namespace)" scope="global" />
   <xacro:property name="namespace" value="$(arg namespace)" scope="global" />
@@ -91,8 +87,8 @@
     <!-- sonar_enabled -->
       <xacro:if value="$(arg sonar_enabled)">
-    <xacro:sonar name="sonar_sensor" x="1.6" y="0.4" z="0.6" ros_topic="/distance1" Y="${radians(0)}"  update_rate="10" min_range="0.3" max_range="2" field_of_view="56" ray_count="2" />
-    <xacro:sonar name="sonar_sensor2" x="1.6" y="-0.4" z="0.6" ros_topic="/distance2" Y="${radians(0)}" update_rate="10" min_range="0.3" max_range="2" field_of_view="56" ray_count="2" />
-    <xacro:sonar name="sonar_sensor3" x="0.3" y="0.4" z="0.6" ros_topic="/distance3" Y="${radians(180)}" update_rate="10" min_range="0.3" max_range="2" field_of_view="56" ray_count="2" />
-    <xacro:sonar name="sonar_sensor4" x="0.3" y="-0.4" z="0.6" ros_topic="/distance4" Y="${radians(180)}" update_rate="10" min_range="0.3" max_range="2" field_of_view="56" ray_count="2" />
+    <xacro:sonar name="sonar_sensor" x="1.6" y="0.4" z="1.6" ros_topic="/distance1" Y="${radians(0)}"  update_rate="10" min_range="0.3" max_range="2" field_of_view="56" ray_count="2" />
+    <xacro:sonar name="sonar_sensor2" x="1.6" y="-0.4" z="1.6" ros_topic="/distance2" Y="${radians(0)}" update_rate="10" min_range="0.3" max_range="2" field_of_view="56" ray_count="2" />
+    <xacro:sonar name="sonar_sensor3" x="0.3" y="0.4" z="1.6" ros_topic="/distance3" Y="${radians(180)}" update_rate="10" min_range="0.3" max_range="2" field_of_view="56" ray_count="2" />
+    <xacro:sonar name="sonar_sensor4" x="0.3" y="-0.4" z="1.6" ros_topic="/distance4" Y="${radians(180)}" update_rate="10" min_range="0.3" max_range="2" field_of_view="56" ray_count="2" />
   </xacro:if>
     <!-- Add CPU Cases -->
@@ -102,19 +98,15 @@
   <!-- Otherwise, add sensors based on enable variables -->
   <xacro:unless value="$(arg yaml_component_generation)">
-    <!-- Add a front camera
-    <xacro:if value="$(arg camera_enabled)">
-      <xacro:wamv_camera name="front_camera" y="0" x="1.5" z="0.65" P="${radians(-20)}" />
-    </xacro:if>-->
     <!-- Add simulated GPS -->
     <xacro:if value="$(arg gps_enabled)">
-      <xacro:wamv_gps name="gps_wamv" x="0.4" y="0" z="0.55" />
+      <xacro:wamv_gps name="gps_wamv" x="0.65" y="-0.1" z="0.55" />
     </xacro:if>
     <!-- Add Simulated IMU -->
     <xacro:if value="$(arg imu_enabled)">
-      <xacro:wamv_imu name="imu_wamv" y="-0.2" />
+      <xacro:wamv_imu name="imu_wamv" x="1.2" y="-0.1" z="0.55" />
     </xacro:if>
     <!-- Add 3D LIDAR -->
     <xacro:if value="$(arg lidar_enabled)">
-      <xacro:lidar name="lidar_wamv" x="0.8" y="0" z="0.7" type="16_beam"/>
+      <xacro:lidar name="lidar_wamv" x="0.6" y="-0.1" z="1.1" type="16_beam"/>
     </xacro:if>
       <!-- Add PLANAR -->
@@ -122,23 +114,10 @@
     	<xacro:wamv_multibeam_laser name="planar_wamv" x="1.2" y="0" z="1"/>
   	</xacro:if>
-    <!-- Add P3D ground truth -->
-    <xacro:if value="$(arg ground_truth_enabled)">
-      <xacro:wamv_p3d name="p3d_wamv"/>
-    </xacro:if>
-    <!-- Add pinger -->
-    <xacro:if value="$(arg pinger_enabled)">
-      <xacro:wamv_pinger name="pinger" position="1.0 0 -1.0" />
-    </xacro:if>
     <!-- ==== VRX sensor configuration ==== -->
     <xacro:if value="$(arg vrx_sensors_enabled)">
-      <!-- Add CPU Cases -->
-      <xacro:include filename="$(find wamv_description)/urdf/cpu_cases.xacro" />
-      <xacro:cpu_cases position="0.75 0 0.65" orientation="0 0 0"/>
-      <!-- Add a stereo camera pair -->
-     <!-- <xacro:wamv_camera name="front_left_camera" y="0.1" x="0.75" P="${radians(15)}" />-->
-      <!--<xacro:wamv_camera name="front_right_camera" y="-0.1" x="0.75" P="${radians(15)}" />-->
       <!-- Add a camera facing right -->
       <xacro:if value="$(arg camera_enabled)">
-      <xacro:wamv_camera name="middle_right_camera" y="0" x="1.5" z="0.65" />
+      <xacro:wamv_camera name="front_camera" y="-0.1" x="1.6" z="1.1" />
+      <xacro:wamv_camera name="back_camera" y="-0.1" x="0.30" z="1.1" P="${radians(-180)}"/>
     </xacro:if>
     </xacro:if>
