Commit message: commit inicial

File: wamv_description/urdf/wamv_base.urdf(original).xacro (robot description, xacro)
@@ -3,40 +3,5 @@
   <!-- Macro for creating the main collisions as simple shapes. -->
   <xacro:macro name="main_collisions" params="prefix reflect:=1">
-<!-- Top part -->
-    <collision name="topPart">
-      <origin xyz="0.95 0.0 0.5"/>
-      <geometry>
-        <box size="1.5 1.1 0.12"/>
-      </geometry>
-    </collision>
-    <!-- External sides -->
-    <collision name="${prefix}_externalSide">
-      <origin xyz="${0.95-0.05} ${((0.5-0.06875)*reflect)} ${0.5-0.29}"/>
-      <geometry>
-        <box size="1.35 0.13 0.67"/>
-      </geometry>
-    </collision>
-    <!-- Internal sides -->
-    <collision name="$prefix_internalSide">
-      <origin xyz="${0.95-0.05} ${((0.446875-0.06875-0.065)*reflect)} ${0.5-0.25}"/>
-      <geometry>
-        <box size="1.35 0.15625 0.5"/>
-      </geometry>
-    </collision>
-   <!-- Center part -->
-    <collision name="centerPart">
-      <origin xyz="${0.95-0.6125} 0.0 ${0.5-0.25}"/>
-      <geometry>
-        <box size="0.20 0.5 0.5"/>
-      </geometry>
-    </collision>
-   <!-- Botoom part -->
-    <collision name="bottomPart">
-      <origin xyz="0.95 0.0 ${0.5-0.25-0.365}"/>
-      <geometry>
-        <box size="1.3 0.55 0.285"/>
-      </geometry>
-    </collision>
-    <!-- Main float
+    <!-- Main float -->
     <collision name="${prefix}_float">
       <origin xyz="-0.4 ${1.03*reflect} 0.2" rpy="${0*reflect} 1.57 0" />
@@ -57,5 +22,5 @@
       </geometry>
     </collision>
-     Front beam
+    <!-- Front beam -->
     <collision name="front_${prefix}_beam_lower">
       <origin xyz="0.9 ${0.85*reflect} 1" rpy="${0.78*reflect} 0 0" />
@@ -70,5 +35,5 @@
       </geometry>
     </collision>
-     Mid beam
+    <!-- Mid beam -->
     <collision name="mid_${prefix}_beam_lower">
       <origin xyz="-0.65 ${0.99*reflect} 0.7" rpy="${0.1*reflect} 0.25 0" />
@@ -89,5 +54,5 @@
       </geometry>
     </collision>
-     Rear beam
+    <!-- Rear beam -->
     <collision name="rear_${prefix}_beam_lower">
       <origin xyz="-0.74 ${1.03*reflect} 0.7" rpy="${0*reflect} -0.15 0" />
@@ -108,5 +73,4 @@
       </geometry>
     </collision>
--->
     <!-- Joint
     <collision name="${prefix}_joint">

File: wamv_gazebo/urdf/components/sonar_sensor(original).xacro (robot description, xacro)
@@ -66,4 +66,8 @@
       </sensor>
     </gazebo>
+    <!-- Set color of post -->
+    <gazebo reference="${name}_link">
+      <material>Gazebo/Black</material>
+    </gazebo>
   </xacro:macro>
 </robot>

File: wamv_gazebo/urdf/components/sonar_sensor(test).xacro (robot description, xacro)
@@ -1,8 +1,8 @@
 <?xml version="1.0"?>
 <robot xmlns:xacro="http://ros.org/wiki/xacro">
-  <xacro:macro name="sonar" params="name x y z R:=0 P:=0 Y:=0 ros_topic update_rate min_range max_range field_of_view ray_count">
+  <xacro:macro name="sonar_sensor" params="name parent *origin ros_topic update_rate min_range max_range field_of_view ray_count">
     <joint name="${name}_joint" type="fixed">
-      <origin xyz= "${x} ${y} ${z}" rpy="${R} ${P} ${Y}" />
-      <parent link="base_link"/>
+      <xacro:insert_block name="origin" />
+      <parent link="${parent}"/>
       <child link="${name}_link"/>
     </joint>
@@ -16,11 +16,6 @@
         <origin xyz="0 0 0" rpy="0 0 0" />
         <geometry>
-          <box size="0.05 0.05 0.05" />
-        </geometry>
-      </visual>
-      <visual>
-        <origin xyz="0.05 0 0" rpy="0 1.57 ${Y}" />
-        <geometry>
-          <cylinder length="0.06" radius="0.02" />
+          <!--<box size="0.01 0.01 0.01" /> -->
+          <mesh filename="package://hector_sensors_description/meshes/sonar_sensor/max_sonar_ez4.dae"/>
         </geometry>
       </visual>
@@ -28,5 +23,5 @@
         <origin xyz="0 0 0" rpy="0 0 0" />
         <geometry>
-          <box size="0.05 0.05 0.05" />
+          <box size="0.01 0.01 0.01" />
         </geometry>
       </collision>
@@ -44,5 +39,5 @@
               <resolution>1</resolution>
               <min_angle>-${field_of_view/2}</min_angle>
-              <max_angle>${field_of_view/2}</max_angle>
+              <max_angle> ${field_of_view/2}</max_angle>
             </horizontal>
             <vertical>
@@ -50,5 +45,5 @@
               <resolution>1</resolution>
               <min_angle>-${field_of_view/2}</min_angle>
-              <max_angle>${field_of_view/2}</max_angle>
+              <max_angle> ${field_of_view/2}</max_angle>
             </vertical>
           </scan>

File: wamv_gazebo/urdf/wamv_gazebo.urdf (original).xacro (robot description, xacro)
@@ -100,17 +100,17 @@
     <!-- Add simulated GPS -->
     <xacro:if value="$(arg gps_enabled)">
-      <xacro:wamv_gps name="gps_wamv" x="0.65" y="0" z="0.3" />
+      <xacro:wamv_gps name="gps_wamv" x="0.65" y="-0.1" z="0.55" />
     </xacro:if>
     <!-- Add Simulated IMU -->
     <xacro:if value="$(arg imu_enabled)">
-      <xacro:wamv_imu name="imu_wamv" x="1.2" y="0" z="0.3" />
+      <xacro:wamv_imu name="imu_wamv" x="1.2" y="-0.1" z="0.55" />
     </xacro:if>
     <!-- Add 3D LIDAR -->
     <xacro:if value="$(arg lidar_enabled)">
-      <xacro:lidar name="lidar_wamv" x="0.6" y="0" z="0.65" type="16_beam"/>
+      <xacro:lidar name="lidar_wamv" x="0.6" y="-0.1" z="1.1" type="16_beam"/>
     </xacro:if>
       <!-- Add PLANAR -->
   	<xacro:if value="$(arg planar_enabled)">
-    	<xacro:wamv_multibeam_laser name="planar_wamv" x="0.6" y="0" z="0.65"/>
+    	<xacro:wamv_multibeam_laser name="planar_wamv" x="1.2" y="0" z="1"/>
   	</xacro:if>
     <!-- ==== VRX sensor configuration ==== -->
@@ -118,6 +118,6 @@
       <!-- Add a camera facing right -->
       <xacro:if value="$(arg camera_enabled)">
-      <xacro:wamv_camera name="front_camera" y="0" x="1.6" z="0.65" />
-      <xacro:wamv_camera name="back_camera" y="0" x="0.30" z="0.65" P="${radians(-180)}"/>
+      <xacro:wamv_camera name="front_camera" y="-0.1" x="1.6" z="1.1" />
+      <xacro:wamv_camera name="back_camera" y="-0.1" x="0.30" z="1.1" P="${radians(-180)}"/>
     </xacro:if>
     </xacro:if>
